File: tegnebrett/getting-started.kicad_pcb (KiCad board)
At the start: 2 copper layers, 199 parts, among them J1 FH12-45S-0.5SH55, J2 FH12-6S-1SH55, J3 Conn_ST_STDC14, J4 DA15_Socket, J5 MCU_Header_Pin, J6 FPGA_Header_Pin, J7 PJ-002A, J8 USB-A1HSW6, J9 FPGA_debug1, SW1 SW_Push, SW2 SW_Push, SW3 Undo, SW4 Reset, SW5 MCU_Button, SW6 FPGA_Button, U1 XC7A100T-2FTG256I, U2 Oscillator 100MHz, U3 TPS54294PWP1, U4 TPS54294PWP2, U5 STM32U5G7VJTxQ, U6 VGA Transceiver, U7 VGA Transciever, U8 IS66WVH16M8DBLL-100B1LI1, Y1 48MHz

Commit message: feat: add footprint to jumper and import to PCB
Parts:
- added JP1: Jumper_2_Open, Connector_PinHeader_2.54mm:PinHeader_1x02_P2.54mm_Vertical, F.Cu at (143.2, 97.0)
- added JP2: Jumper_2_Open, Connector_PinHeader_2.54mm:PinHeader_1x02_P2.54mm_Vertical, F.Cu at (147.8, 97.0)
- added JP3: Jumper_2_Open, Connector_PinHeader_2.54mm:PinHeader_1x02_P2.54mm_Vertical, F.Cu at (152.4, 97.0)
- added JP4: Jumper_2_Open, Connector_PinHeader_2.54mm:PinHeader_1x02_P2.54mm_Vertical, F.Cu at (157.0, 97.0)
Connections:
- C101 pad 1: +3V3 -> Net-(JP3-A)
- C102 pad 1: +5V -> Net-(JP4-A)
- C103 pad 1: +5V -> Net-(JP4-A)
- C20 pad 1: +3V3 -> Net-(JP3-A)
- C91 pad 1: +1V0 -> Net-(JP1-A)
- C92 pad 1: +1V0 -> Net-(JP1-A)
- C95 pad 1: +1V8 -> Net-(JP2-A)
- C96 pad 1: +1V8 -> Net-(JP2-A)
- L5 pad 1: +1V0 -> Net-(JP1-A)
- L6 pad 1: +1V8 -> Net-(JP2-A)
- L7 pad 1: +3V3 -> Net-(JP3-A)
- L8 pad 1: +5V -> Net-(JP4-A)
- R15 pad 2: +3V3 -> Net-(JP3-A)
- R80 pad 1: +1V0 -> Net-(JP1-A)
- R83 pad 1: +1V8 -> Net-(JP2-A)
- R86 pad 1: +3V3 -> Net-(JP3-A)
- R88 pad 1: +5V -> Net-(JP4-A)

Commit message: pcb: update from schematic
reloads the annotations used.
Parts:
- renumbered C71 to C1, C80 to C10, C82 to C11, C81 to C12, C84 to C13, C83 to C14, C85 to C15, C86 to C16, C46 to C17, C47 to C18, C48 to C19, C72 to C2, C49 to C20, C50 to C21, C51 to C22, C87 to C23, C88 to C24, C89 to C25, C90 to C26, C1 to C27, C3 to C28, C4 to C29, C73 to C3, C5 to C30, C6 to C31, C7 to C32, C9 to C33, C10 to C34, C11 to C35, C12 to C36, C13 to C37, C15 to C38, C16 to C39, C74 to C4, C17 to C40, C18 to C41, C19 to C42, C21 to C43, C22 to C44, C23 to C45, C24 to C46, C26 to C47, C27 to C48, C28 to C49, C75 to C5, C29 to C50, C31 to C51, C32 to C52, C33 to C53, C34 to C54, C36 to C55, C37 to C56, C38 to C57, C39 to C58, C40 to C59, C76 to C6, C41 to C60, C42 to C61, C43 to C62, C44 to C63, C45 to C64, C92 to C65, C20 to C66, C91 to C67, C101 to C68, C8 to C69, C77 to C7, C2 to C70, C25 to C71, C98 to C72, C35 to C73, C104 to C74, C93 to C75, C94 to C76, C105 to C77, C97 to C78, C100 to C79, C79 to C8, C14 to C80, C99 to C81, C30 to C82, C103 to C83, C96 to C84, C102 to C85, C95 to C86, C78 to C9, D8 to D1, D9 to D2, D2 to D3, D3 to D4, D1 to D5, J8 to J4, J9 to J6, J6 to J7, J4 to J8, J7 to J9, JP3 to JP2, JP4 to JP3, JP2 to JP4, L4 to L1, L5 to L2, L7 to L3, L8 to L4, L6 to L5, R17 to R1, R79 to R10, R9 to R11, R10 to R12, R11 to R13, R12 to R14, R1 to R15, R2 to R16, R3 to R17, R4 to R18, R5 to R19, R18 to R2, R6 to R20, R7 to R21, R8 to R22, R64 to R23, R22 to R24, R72 to R25, R73 to R26, R14 to R27, R23 to R28, R24 to R29, R19 to R3, R25 to R30, R26 to R31, R27 to R32, R28 to R33, R29 to R34, R30 to R35, R31 to R36, R32 to R37, R33 to R38, R34 to R39, R20 to R4, R35 to R40, R36 to R41, R37 to R42, R38 to R43, R39 to R44, R40 to R45, R41 to R46, R42 to R47, R43 to R48, R44 to R49, R21 to R5, R45 to R50, R46 to R51, R47 to R52, R48 to R53, R49 to R54, R50 to R55, R51 to R56, R52 to R57, R53 to R58, R54 to R59, R78 to R6, R55 to R60, R56 to R61, R57 to R62, R58 to R63, R59 to R64, R60 to R65, R61 to R66, R62 to R67, R15 to R68, R80 to R69, R63 to R7, R81 to R70, R86 to R71, R87 to R72, R82 to R73, R85 to R74, R88 to R75, R89 to R76, R83 to R77, R84 to R78, R13 to R8, R65 to R9, SW5 to SW3, SW3 to SW5, U5 to U1, U1 to U2, U2 to U3, U8 to U4, U6 to U5, U7 to U6, U4 to U7, U3 to U8
