File: tegnebrett/FPGA.kicad_sch (KiCad schematic)
At the start: 28 parts, among them J6 FPGA_debug, J7 FPGA_Header_Pin, SW6 FPGA_Button, U2 XC7A100T-2FTG256I, U3 Oscillator 100MHz, U4 IS66WVH16M8DBLL-100B1LI1

Commit message: fix: Save FPGA SRAM symbol to tegnebrett_symbols.kicad_sch
And update symbol in the FPGA.kicad_sch sheet.
Removes one warning.
Parts:
- U4: symbol XC7A100T-2FTG256I:IS66WVH16M8DBLL-100B1LI -> tegnebrett_symbols:IS66WVH16M8DBLL-100B1LI
Changed lines of the file:
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@@
 	)
 	(symbol
-		(lib_id "XC7A100T-2FTG256I:IS66WVH16M8DBLL-100B1LI")
+		(lib_id "tegnebrett_symbols:IS66WVH16M8DBLL-100B1LI")
 		(at 363.22 96.52 0)
 		(unit 1)

Commit message: refactor: move FPGA button from g12 to a13 pin on FPGA
g12 -> a13
This makes the routing easier.
Connections:
- net at U2.A13 (IO_L7P_T1_AD2P_15): now also R27.2, SW6.1
- now unconnected: U2.G12 (IO_L19N_T3_A21_VREF_15)
Other:
- moved on the sheet: R27, SW6
Changed lines of the file:
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@@
 	)
 	(junction
+		(at 341.63 71.12)
+		(diameter 0)
+		(color 0 0 0 0)
+	)
+	(junction
 		(at 144.78 49.53)
 		(diameter 0)
@@
 	)
 	(junction
-		(at 334.01 144.78)
-		(diameter 0)
-		(color 0 0 0 0)
-	)
-	(junction
 		(at 86.36 29.21)
 		(diameter 0)
@@
 	)
 	(no_connect
-		(at 320.04 81.28)
-	)
-	(no_connect
 		(at 16.51 198.12)
 	)
@@
 	)
 	(no_connect
+		(at 320.04 144.78)
+	)
+	(no_connect
 		(at 118.11 205.74)
 	)
@@
 	(wire
 		(pts
+			(xy 320.04 81.28) (xy 336.55 81.28)
+		)
+		(stroke
+			(width 0)
+			(type default)
+		)
+	)
+	(wire
+		(pts
 			(xy 86.36 29.21) (xy 101.6 29.21)
 		)
@@
 	(wire
 		(pts
-			(xy 334.01 144.78) (xy 337.82 144.78)
+			(xy 341.63 71.12) (xy 345.44 71.12)
 		)
 		(stroke
@@
 	(wire
 		(pts
+			(xy 336.55 71.12) (xy 341.63 71.12)
+		)
+		(stroke
+			(width 0)
+			(type default)
+		)
+	)
+	(wire
+		(pts
 			(xy 107.95 68.58) (xy 107.95 71.12)
 		)
@@
 	(wire
 		(pts
-			(xy 132.08 60.96) (xy 173.99 60.96)
+			(xy 336.55 81.28) (xy 336.55 71.12)
 		)
 		(stroke
@@
 	(wire
 		(pts
-			(xy 208.28 83.82) (xy 208.28 93.98)
+			(xy 132.08 60.96) (xy 173.99 60.96)
 		)
 		(stroke
@@
 	(wire
 		(pts
-			(xy 85.09 58.42) (xy 96.52 58.42)
+			(xy 208.28 83.82) (xy 208.28 93.98)
 		)
 		(stroke
@@
 	(wire
 		(pts
-			(xy 320.04 144.78) (xy 334.01 144.78)
+			(xy 85.09 58.42) (xy 96.52 58.42)
 		)
 		(stroke
@@
 	(symbol
 		(lib_id "power:+3V3")
-		(at 334.01 137.16 0)
+		(at 341.63 63.5 0)
 		(unit 1)
 		(exclude_from_sim no)
@@
 		(dnp no)
 		(property "Reference" "#PWR035"
-			(at 334.01 140.97 0)
+			(at 341.63 67.31 0)
 			(effects
 				(font
@@
 		)
 		(property "Value" "+3V3"
-			(at 336.55 135.636 0)
+			(at 344.17 61.976 0)
 			(effects
 				(font
@@
 		)
 		(property "Footprint" ""
-			(at 334.01 137.16 0)
+			(at 341.63 63.5 0)
 			(effects
 				(font
@@
 		)
 		(property "Datasheet" ""
-			(at 334.01 137.16 0)
+			(at 341.63 63.5 0)
 			(effects
 				(font
@@
 		)
 		(property "Description" "Power symbol creates a global label with name \"+3V3\""
-			(at 334.01 137.16 0)
+			(at 341.63 63.5 0)
 			(effects
 				(font
@@
 	(symbol
 		(lib_id "power:GND")
-		(at 347.98 144.78 90)
+		(at 355.6 71.12 90)
 		(unit 1)
 		(exclude_from_sim no)
@@
 		(fields_autoplaced yes)
 		(property "Reference" "#PWR038"
-			(at 354.33 144.78 0)
+			(at 361.95 71.12 0)
 			(effects
 				(font
@@
 		)
 		(property "Value" "GND"
-			(at 351.79 144.7799 90)
+			(at 359.41 71.1199 90)
 			(effects
 				(font
@@
 		)
 		(property "Footprint" ""
-			(at 347.98 144.78 0)
+			(at 355.6 71.12 0)
 			(effects
 				(font
@@
 		)
 		(property "Datasheet" ""
-			(at 347.98 144.78 0)
+			(at 355.6 71.12 0)
 			(effects
 				(font
@@
 		)
 		(property "Description" "Power symbol creates a global label with name \"GND\" , ground"
-			(at 347.98 144.78 0)
+			(at 355.6 71.12 0)
 			(effects
 				(font
@@
 	(symbol
 		(lib_id "Switch:SW_Push")
-		(at 342.9 144.78 0)
+		(at 350.52 71.12 0)
 		(unit 1)
 		(exclude_from_sim no)
@@
 		(dnp no)
 		(property "Reference" "SW6"
-			(at 342.9 147.066 0)
+			(at 350.52 73.406 0)
 			(effects
 				(font
@@
 		)
 		(property "Value" "FPGA_Button"
-			(at 343.154 141.478 0)
+			(at 350.774 67.818 0)
 			(effects
 				(font
@@
 		)
 		(property "Footprint" "tegnebrett_modules:SW_PS1024ALRED"
-			(at 342.9 139.7 0)
+			(at 350.52 66.04 0)
 			(effects
 				(font
@@
 		)
 		(property "Datasheet" "~"
-			(at 342.9 139.7 0)
+			(at 350.52 66.04 0)
 			(effects
 				(font
@@
 		)
 		(property "Description" "Push button switch, generic, two pins"
-			(at 342.9 144.78 0)
+			(at 350.52 71.12 0)
 			(effects
 				(font
@@
 	(symbol
 		(lib_id "Device:R")
-		(at 334.01 140.97 0)
+		(at 341.63 67.31 0)
 		(unit 1)
 		(exclude_from_sim no)
@@
 		(dnp no)
 		(property "Reference" "R27"
-			(at 334.01 137.414 0)
+			(at 341.63 63.754 0)
 			(effects
 				(font
@@
 		)
 		(property "Value" "4.7k"
-			(at 334.01 142.748 90)
+			(at 341.63 69.088 90)
 			(effects
 				(font
@@
 		)
 		(property "Footprint" "Resistor_SMD:R_0805_2012Metric_Pad1.20x1.40mm_HandSolder"
-			(at 332.232 140.97 90)
+			(at 339.852 67.31 90)
 			(effects
 				(font
@@
 		)
 		(property "Datasheet" "~"
-			(at 334.01 140.97 0)
+			(at 341.63 67.31 0)
 			(effects
 				(font
@@
 		)
 		(property "Description" "Resistor"
-			(at 334.01 140.97 0)
+			(at 341.63 67.31 0)
 			(effects
 				(font
