File: tegnebrett/FPGA.kicad_sch (KiCad schematic)
At the start: 28 parts, among them J6 FPGA_debug, J7 FPGA_Header_Pin, SW6 FPGA_Button, U2 XC7A100T-2FTG256I, U3 Oscillator 100MHz, U4 IS66WVH16M8DBLL-100B1LI1

Commit message: fix: add project-local variant of FPGA symbol
Allows us to set some bi-directional pins to *power input*, as some of
the bi-directionals are connected to GND and VDD. KiCAD threw warning
because of that.
Now the warning count is down to 1.
Parts:
- U2: symbol FPGA_Xilinx_Artix7:XC7A100T-FTG256 -> tegnebrett_symbols:XC7A100T-FTG256
Changed lines of the file:
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@@
 	)
 	(symbol
-		(lib_id "FPGA_Xilinx_Artix7:XC7A100T-FTG256")
+		(lib_name "XC7A100T-FTG256_1")
+		(lib_id "tegnebrett_symbols:XC7A100T-FTG256")
 		(at 269.24 101.6 0)
 		(unit 1)
@@
 	)
 	(symbol
-		(lib_id "FPGA_Xilinx_Artix7:XC7A100T-FTG256")
+		(lib_name "XC7A100T-FTG256_2")
+		(lib_id "tegnebrett_symbols:XC7A100T-FTG256")
 		(at 67.31 205.74 0)
 		(unit 2)
@@
 	)
 	(symbol
-		(lib_id "FPGA_Xilinx_Artix7:XC7A100T-FTG256")
+		(lib_id "tegnebrett_symbols:XC7A100T-FTG256")
 		(at 46.99 73.66 0)
 		(unit 3)
