File: tegnebrett/VGA.kicad_sch (KiCad schematic)
At the start: 47 parts, among them J8 DA15_Socket, U5 VGA Transceiver, U6 VGA Transciever

Commit message: fix: Add separate symbol for second VGA-transceiver
Some pins are bi-directional on the one symbol, but grounded on the
other. This new symbol and subsequent update to schematic symbol reduces
the warning count by 2.
Parts:
- U6: symbol tegnebrett_symbols:SN74ALVC245PWR -> tegnebrett_symbols:SN74ALVC245PWR-extra-GND
Changed lines of the file:
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@@
 	)
 	(symbol
-		(lib_id "tegnebrett_symbols:SN74ALVC245PWR")
+		(lib_id "tegnebrett_symbols:SN74ALVC245PWR-extra-GND")
 		(at 78.74 128.27 0)
 		(unit 1)
