File: tegnebrett/Power_FPGA.kicad_sch (KiCad schematic)
At the start: 39 parts, among them U2 XC7A100T-2FTG256I

Commit message: fix: add project-local variant of FPGA symbol
Allows us to set some bi-directional pins to *power input*, as some of
the bi-directionals are connected to GND and VDD. KiCAD threw warning
because of that.
Now the warning count is down to 1.
Parts:
- U2: symbol FPGA_Xilinx_Artix7:XC7A100T-FTG256 -> tegnebrett_symbols:XC7A100T-FTG256
Changed lines of the file:
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@@
 	)
 	(symbol
-		(lib_id "FPGA_Xilinx_Artix7:XC7A100T-FTG256")
+		(lib_id "tegnebrett_symbols:XC7A100T-FTG256")
 		(at 204.47 85.09 0)
 		(unit 4)
